Commit message: new stuff

File: src/description_pkg/urdf/uic_bot.xacro (robot description, xacro)
@@ -179,5 +179,6 @@
     <parent link="base_link" />
     <child link="d455_link" />
-    <origin xyz="-0.42 0 0.37" rpy="0 0.523599 3.14" />
+    <origin xyz="-0.556 0.032 0.464" rpy="0 0 3.14159" />
+    <!-- Note: rpy has yaw=π (180°) to face backward, pitch=25° down = 0.436 rad -->
   </joint>
   <joint name="d455_optical_joint" type="fixed">
@@ -189,5 +190,5 @@
     <parent link="base_link" />
     <child link="d456_link" />
-    <origin xyz="0.535 -0.28 0.141" rpy="0 0 0" />
+    <origin xyz="0.457 -0.289 0.210" rpy="0 0 0" />
   </joint>
   <joint name="d456_optical_joint" type="fixed">
@@ -199,5 +200,5 @@
     <parent link="base_link" />
     <child link="s3_lidar_link" />
-    <origin xyz="-0.38 -0.0889 0.2811" rpy="0 0 0" />
+    <origin xyz="-0.38 0.102 0.470" rpy="0 0 0"/>
   </joint>
   <joint name="imu_joint" type="fixed">

Commit message: simwork

File: src/description_pkg/urdf/uic_bot.xacro (robot description, xacro)
@@ -179,6 +179,5 @@
     <parent link="base_link" />
     <child link="d455_link" />
-    <origin xyz="-0.556 0.032 0.464" rpy="0 0 3.14159" />
-    <!-- Note: rpy has yaw=π (180°) to face backward, pitch=25° down = 0.436 rad -->
+    <origin xyz="-0.42 0 0.37" rpy="0 0.523599 3.14" />
   </joint>
   <joint name="d455_optical_joint" type="fixed">
@@ -190,5 +189,5 @@
     <parent link="base_link" />
     <child link="d456_link" />
-    <origin xyz="0.457 -0.289 0.210" rpy="0 0 0" />
+    <origin xyz="0.535 -0.28 0.141" rpy="0 0 0" />
   </joint>
   <joint name="d456_optical_joint" type="fixed">
@@ -200,5 +199,5 @@
     <parent link="base_link" />
     <child link="s3_lidar_link" />
-    <origin xyz="-0.38 0.102 0.470" rpy="0 0 0"/>
+    <origin xyz="-0.38 -0.0889 0.2811" rpy="0 0 0" />
   </joint>
   <joint name="imu_joint" type="fixed">

Commit message: new

File: src/description_pkg/urdf/uic_bot.xacro (robot description, xacro)
@@ -47,5 +47,5 @@
         <mesh filename="file:///$(find description_pkg)/meshes/uic_bot/d456_camera.stl" />
       </geometry>
-      <origin xyz="0 -${camera_sim_link_offset} 0" rpy="0 0 0" />
+    <!--  <origin xyz="0 -${camera_sim_link_offset} 0" rpy="0 0 0" /> -->
       <material name="camera_grey" />
     </visual>
@@ -54,5 +54,5 @@
         <mesh filename="file:///$(find description_pkg)/meshes/uic_bot/d456_camera.stl" />
       </geometry>
-      <origin xyz="0 -${camera_sim_link_offset} 0" rpy="0 0 0" />
+    <!--  <origin xyz="0 -${camera_sim_link_offset} 0" rpy="0 0 0" /> -->
     </collision>
   </link>
@@ -63,5 +63,5 @@
         <mesh filename="file:///$(find description_pkg)/meshes/uic_bot/d455_camera.stl" />
       </geometry>
-      <origin xyz="0 -${camera_sim_link_offset} 0" rpy="0 0 0" />
+    <!--  <origin xyz="0 -${camera_sim_link_offset} 0" rpy="0 0 0" /> -->
       <material name="camera_grey" />
     </visual>
@@ -70,5 +70,5 @@
         <mesh filename="file:///$(find description_pkg)/meshes/uic_bot/d455_camera.stl" />
       </geometry>
-      <origin xyz="0 -${camera_sim_link_offset} 0" rpy="0 0 0" />
+    <!--  <origin xyz="0 -${camera_sim_link_offset} 0" rpy="0 0 0" /> -->
     </collision>
   </link>
@@ -179,5 +179,5 @@
     <parent link="base_link" />
     <child link="d455_link" />
-    <origin xyz="-0.42 0 0.37" rpy="0 0.523599 3.14" />
+    <origin xyz="-0.42 0 0.37" rpy="0 -0.2618 3.14" />
   </joint>
   <joint name="d455_optical_joint" type="fixed">
@@ -189,5 +189,5 @@
     <parent link="base_link" />
     <child link="d456_link" />
-    <origin xyz="0.535 -0.28 0.141" rpy="0 0 0" />
+    <origin xyz="0.535 -0.28 0.141" rpy="0 -0.2618 0" />
   </joint>
   <joint name="d456_optical_joint" type="fixed">
@@ -199,5 +199,5 @@
     <parent link="base_link" />
     <child link="s3_lidar_link" />
-    <origin xyz="-0.38 -0.0889 0.2811" rpy="0 0 0" />
+    <origin xyz="0.0 0.102 0.470" rpy="0 0 0" />
   </joint>
   <joint name="imu_joint" type="fixed">
